File: Geiger_v4.brd (EAGLE design)
At the start: 112.4 x 60.5 mm, 126 parts, among them J1 01010002Z, J2 USB4085-GF-A, J3 01010002Z, J4 01010002Z, J5 01010002Z, Q1 MMBT3904, Q2 MMBT3904, Q3 PMBTA45,215, Q4 MMBT3904, Q5 MMBT3904, Q6 MMBT3904, Q7 AO3400A, Q8 AO3400A, SW1 SPDT, U1 TLC555CDR, U2 FM2113, U3 ESP32-WROOM-32D-N8, U4 CP2102N-A01-GQFN28, U6 TPS63000DRCR, U7 LP28013A

Commit message: release
Parts:
- added R54, R55, R9: 10, ruark2:0603
- moved J4 5.08 mm to (89.3, 43.0)
- moved J5 2.27 mm to (60.5, 43.0)
- moved C19 0.76 mm to (89.5, 29.5)
- moved C3 0.76 mm to (89.5, 23.4)
- moved C4 0.76 mm to (89.5, 27.5)
- moved C5 0.76 mm to (89.5, 25.4)
Connections:
- new net N$56: R50.3, R54.2, R55.2, R9.1
- net GND: now also R54.1, R55.1, U7.4; no longer R50.3
- net N$11: now also R9.2
- net VUSBIN: no longer U7.4
Routing:
- net N$56: track 0.00 -> 9.16 mm
- net N$11: track 14.2 -> 20.7 mm
- net N$40: track 36.0 -> 33.2 mm
- net N$15: track 17.1 -> 14.3 mm
- net N$53: track 41.2 -> 38.9 mm
- net GND: track 2.73 -> 4.31 mm, vias 109 -> 112
- net VUSBIN: track 51.6 -> 50.7 mm
- net N$35: track 46.2 -> 45.5 mm
Other:
- board text added: "003"
- board text added: "10"
- board text added: "20"
- board text added: "30"
- board text added: "40"
- board text added: "60"
- board text added: "70"
- board text added: "90"
- board text added: "MMXXIV"
- board text removed: "062"
- board text removed: "MMXXIII"
