File: Geiger_v4.sch (EAGLE design)
At the start: 126 parts, among them J1 01010002Z, J2 USB4085-GF-A, J3 01010002Z, J4 01010002Z, J5 01010002Z, Q1 MMBT3904, Q2 MMBT3904, Q3 PMBTA45,215, Q4 MMBT3904, Q5 MMBT3904, Q6 MMBT3904, Q7 AO3400A, Q8 AO3400A, SW1 SPDT, U1 TLC555CDR, U2 FM2113, U3 ESP32-WROOM-32D-N8, U4 CP2102N-A01-GQFN28, U6 TPS63000DRCR, U7 LP28013A

Commit message: release
Parts:
- added R54, R55, R9: 10, ruark2:0603_RESISTOR
Connections:
- new net N$56: R50.2, R54.2, R55.2, R9.1
- net GND: now also R54.1, R55.1, U7.EN; no longer R50.2
- net N$11: now also R9.2
- net VUSBIN: no longer U7.EN
Other:
- note added: "EN is active low..."
- note added: "JLCPCB Assembly Notes: -Change CP210 part number -Make sure to place 10mH inductor -Check rotation of all rotation sensitive parts."
- note removed: "20k"
- note removed: "47k"
- moved on the sheet: C21, C7, Q2, R1, R14, R50
